Commit message: Update to ROS 2 Jazzy: Modify Dockerfile, launch files, and configuration for compatibility

File: hunter_description/description/meshes.xacro (robot description, xacro)
@@ -11,5 +11,19 @@
       <origin xyz="0 0 0" rpy="0 0 0"/>
       <geometry>
-        <mesh filename="file://$(find hunter_description)/meshes/${name}.dae" />
+        <xacro:if value="${name == 'chassis'}">
+          <box size="0.90 0.60 0.30"/>
+        </xacro:if>
+        <xacro:if value="${name == 'rear_left_wheel'}">
+          <cylinder length="0.07" radius="0.165"/>
+        </xacro:if>
+        <xacro:if value="${name == 'rear_right_wheel'}">
+          <cylinder length="0.07" radius="0.165"/>
+        </xacro:if>
+        <xacro:if value="${name == 'front_left_wheel'}">
+          <cylinder length="0.07" radius="0.165"/>
+        </xacro:if>
+        <xacro:if value="${name == 'front_right_wheel'}">
+          <cylinder length="0.07" radius="0.165"/>
+        </xacro:if>
       </geometry>
     </collision>

File: hunter_description/description/robot_core.xacro (robot description, xacro)
@@ -29,6 +29,6 @@
     <origin xyz="${x_base_to_rear} ${y_base_to_wheel} ${z_base_to_wheel}" rpy="${pi/2} 0 0" />
     <axis xyz="0 0 -1" />
-    <dynamics damping="0.2" friction="15"/>
-    <limit effort="10.0" velocity="10.0"/>
+    <dynamics damping="0.01" friction="0.1"/>
+    <limit effort="100.0" velocity="100.0"/>
   </joint>
   <xacro:gazebo_friction reference="rear_left_wheel"/>
@@ -42,6 +42,6 @@
     <origin xyz="${x_base_to_rear} -${y_base_to_wheel} ${z_base_to_wheel}" rpy="${pi/2} 0 0" />
     <axis xyz="0 0 -1"/>
-    <dynamics damping="0.2" friction="15"/>
-    <limit effort="10.0" velocity="10.0"/>
+    <dynamics damping="0.01" friction="0.1"/>
+    <limit effort="100.0" velocity="100.0"/>
     <!-- <mimic joint="rear_left_wheel_joint" multiplier="1.0" offset="0.0"/> -->
   </joint>

File: hunter_description/description/ros2_control.xacro (robot description, xacro)
@@ -35,4 +35,5 @@
     <plugin filename="libgz_ros2_control-system.so" name="gz_ros2_control::GazeboSimROS2ControlPlugin">
       <parameters>$(find hunter_description)/config/ackermann_like_controller.yaml</parameters>
+      <parameters>$(find hunter_description)/config/gazebo_params.yaml</parameters>
     </plugin>
   </gazebo>
